File: Modulo_Material_particulado.kicad_sch (KiCad schematic)
At the start: 12 parts, among them J1 PMS7003, J2 OLED_iic, J3 BME_280, J4 V_INT, U1 AMS1117-5.0, U2 ESP32-DEVKIT-V1

Commit message: fix: se corrigieron componentes erroneos
Parts:
- removed J4: V_INT, Button_Switch_THT:SW_DIP_SPSTx01_Slide_6.7x4.1mm_W7.62mm_P2.54mm_LowProfile, symbol Connector:Screw_Terminal_01x02
- removed R1, R2: 4700, Button_Switch_THT:SW_DIP_SPSTx01_Slide_6.7x4.1mm_W7.62mm_P2.54mm_LowProfile, symbol Device:R
- removed U2: ESP32-DEVKIT-V1, RF_Module:ESP32-C3-DevKitM-1, symbol ESP32-DEVKIT-V1:ESP32-DEVKIT-V1
- added J5: USB_C_Receptacle_USB2.0_16P, Connector_USB:USB_C_Receptacle_Amphenol_12401948E412A, symbol Connector:USB_C_Receptacle_USB2.0_16P
- added U3: ESP32-S3-WROOM-1, RF_Module:ESP32-S3-WROOM-1, symbol RF_Module:ESP32-S3-WROOM-1
- C1, C6: footprint Capacitor_THT:C_Disc_D3.0mm_W2.0mm_P2.50mm -> Capacitor_SMD:C_0805_2012Metric
- C3, C5: footprint Capacitor_THT:C_Radial_D6.3mm_H11.0mm_P2.50mm -> Capacitor_SMD:C_0805_2012Metric
Connections:
- net 5V: no longer C5.1, C6.1, U1.2 (VO)
- net GND: now also J5.A1 (GND), J5.A12 (GND), J5.B1 (GND), J5.B12 (GND), J5.SH (SHIELD)
- net +5V: now reaches C1.1, C3.1, U1.3 (VI)
- net +5V: now also J5.A4 (VBUS), J5.A9 (VBUS), J5.B4 (VBUS), J5.B9 (VBUS)
- new net: U3.1 (GND), U3.40 (GND), U3.41 (GND)
- new net +3V3: C5.1, C6.1, U1.2 (VO)
- new net D+: J5.A6 (D+), J5.B6 (D+), U3.14 (USB_D+)
- new net D-: J5.A7 (D-), J5.B7 (D-), U3.13 (USB_D-)
Other:
- moved on the sheet: J1, J2, J3
